Commit message: Correct ogm, ego , map not localized
Signed-off-by: Hesam Taherzadegan <Taherzadehesam@gmail.com>

File: src/bev/urdf/robot.urdf (robot description, URDF)
Before this commit: robot kitti_robot, 3 links, 2 joints
Links:
- added link camera_color_left
Joints:
- added joint base_to_camera: type fixed, parent base_link, child camera_color_left, origin xyz=0 0 0.0 rpy=0 0 0
